File: Design/HF091CBU.sch (EAGLE design)
At the start: 40 parts, among them J1 629105136821, U1 STM32F091CBU6, U2 FT232RQ, X1 XTALL_CSTCE8M00G52

Commit message: All finish, reviewed version
Parts:
- removed JP1, JP2: (no value), pinhead:PINHD-1X20
- removed VRJ: (no value), jumper:SJ
- added JP_L, JP_R: (no value), HEXABITZ_USER_INTERFACE_PARTS:PINHD-1X20
- added VBJ: (no value), jumper:SJ
- C1, C11, C12, C13, C14, C15, C17, C5, C6, C7, C8, C9: device Hexabitz:C-0603 -> HEXABITZ_RCLS:C-0603
- C2: device Hexabitz:C-0805-POL -> HEXABITZ_RCLS:C-0805; CAPACITANCE 1.00uF -> (none); MFN Yageo -> (none); MPN CC0805KKX7R7BB105 -> (none); OCTOPART_URL https://octopart.com/cc0805kkx7r7bb105-yageo-8376555?r=sp&s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 -> (none); TOLERANCE 10% -> (none); VOLTAGE_RATING 16V -> (none)
- C3, C4: device Hexabitz:C-0805-POL -> HEXABITZ_RCLS:C-0805; CAPACITANCE 4.7uF -> (none); MFN Murata -> (none); MPN GRM21BC81E475KA12L -> (none); OCTOPART_URL https://octopart.com/grm21bc81e475ka12l-murata-10331911?r=s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 -> (none); TOLERANCE 10% -> (none); VOLTAGE_RATING 25V -> (none)
- FB1, FB2: device Hexabitz:FB-TDK_MMZ1608Y300B -> HEXABITZ_RCLS:FB-0603
- R1, R2, R4, R5: device Hexabitz:R-0603 -> HEXABITZ_RCLS:R-0603
- R3: device Hexabitz:R-0603 -> HEXABITZ_RCLS:R-0603; RESISTANCE 0.0 Ohm -> (none)
- SWD: device pinhead:PINHD-1X5/90 -> HEXABITZ_USER_INTERFACE_PARTS:PINHD-1X5/90
- TRIMBLE-LOGO1: value HEXA-LOGO -> HEXABITZ-LOGO_NO_BOTTOM_SPLIT; device HEXABITZ_USER_INTERFACE_PARTS:HEXA-LOGO -> HEXABITZ_USER_INTERFACE_PARTS:HEXABITZ-LOGO_NO_BOTTOM_SPLIT
Connections:
- removed net N$7: U1.VBAT, VRJ.2
- removed net PA10: JP1.1
- removed net PA13: U1.PA15
- removed net PA9: JP1.2
- removed net PB0: JP1.12, U1.PB0
- removed net PD0: JP2.19
- removed net PD1: JP2.18
- removed net PD2: JP2.17
- removed net PD3: JP2.16
- removed net VREF: JP2.5
- new net PC13: JP_L.7, U1.PC13
- new net PC15: JP_L.9, U1.PC15-OSC32_OUT
- net +5V: now also JP_L.1; no longer JP2.1
- net GND: now also C3.2, C4.2, JP_L.2, JP_L.20; no longer C3.-, C4.-, JP2.2
- net PA0: now also JP_L.10; no longer JP1.20
- net PA1: now also JP_L.11; no longer JP1.19
- net PA11: now also JP_R.10
- net PA12: now also JP_R.9
- net PA15: now also JP_R.8, U1.PA15; no longer JP2.20
- net PA2: now also JP_L.12; no longer JP1.18
- net PA3: now also JP_L.13; no longer JP1.17
- net PA4: now also JP_L.14; no longer JP1.16
- net PA5: now also JP_L.15; no longer JP1.15
- net PA6: now also JP_L.16; no longer JP1.14
- net PA7: now also JP_L.17; no longer JP1.13
- net PA8: now also JP_R.13; no longer JP1.3
- net PB1: now also JP_L.18; no longer JP1.11
- net PB10: now also JP_R.19; no longer JP1.9
- net PB11: now also JP_R.18; no longer JP1.8
- net PB12: now also JP_R.17; no longer JP1.7
- net PB13: now also JP_R.16; no longer JP1.6
- net PB14: now also JP_R.15; no longer JP1.5
- net PB15: now also JP_R.14; no longer JP1.4
- net PB2: now also JP_L.19; no longer JP1.10
- net PB3: now also JP_R.7; no longer JP2.15
- net PB4: now also JP_R.6; no longer JP2.14
- net PB5: now also JP_R.5; no longer JP2.13
- net PB6: now also JP_R.4; no longer JP2.12
- net PB7: now also JP_R.3; no longer JP2.11
- net PB8: now also JP_R.2; no longer JP2.10
- net PB9: now also JP_R.1; no longer JP2.9
- net PC14: now also JP_L.8, U1.PC14-OSC32_IN; no longer JP2.8
- net RX1: now also JP_R.11
- net TX1: now also JP_R.12
- net USER_LED: now also U1.PB0
- net VBAT: now also C9.1, JP_L.4, U1.VBAT, VBJ.2; no longer JP2.6
- net VDD: now also C3.1, C4.1, JP_L.3, JP_R.20, VBJ.1; no longer C3.+, C4.+, C9.1, JP2.3, VRJ.1
- net VDDA: now also C2.1, JP_L.5; no longer C2.+, JP2.4
- net VSSA: now also C2.2, JP_L.6; no longer C2.-, JP2.7
Other:
- note removed: "VBAT"
- moved on the sheet: C17, R3
